File: cpu-2.kicad_sch (KiCad schematic)
At the start: 156 parts, among them Q1 2N2369A, X1 14-Pin Socket, X2 14-Pin Socket, X3 14-Pin Socket, X4 14-Pin Socket, X5 14-Pin Socket, X6 14-Pin Socket

Commit message: Final commit of combined repo before disassociating from combined repos and re-establishing as a standalone repo
Connections:
- net +5V: now also X6.3
- net -12V: now also X6.5
Changed lines of the file:
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@@
     (stroke (width 1) (type default) (color 255 0 0 1))
   )
-  (wire (pts (xy 305.054 64.516) (xy 305.054 60.198))
+  (wire (pts (xy 305.054 65.024) (xy 305.054 60.198))
     (stroke (width 0) (type default))
   )
@@
     (stroke (width 0) (type default))
   )
+  (wire (pts (xy 345.694 48.26) (xy 345.694 51.308))
+    (stroke (width 0) (type default))
+  )
   (wire (pts (xy 300.99 50.038) (xy 312.674 50.038))
     (stroke (width 0) (type default))
@@
     (stroke (width 0) (type default))
   )
-  (wire (pts (xy 210.566 64.516) (xy 305.054 64.516))
+  (wire (pts (xy 210.566 65.024) (xy 305.054 65.024))
     (stroke (width 0) (type default))
   )
@@
     (stroke (width 0) (type default))
   )
-  (wire (pts (xy 210.566 122.174) (xy 210.566 161.036))
+  (wire (pts (xy 210.566 121.92) (xy 210.566 161.036))
     (stroke (width 0) (type default))
   )
@@
     (stroke (width 0) (type default))
   )
-  (wire (pts (xy 210.566 121.92) (xy 210.566 64.516))
-    (stroke (width 0) (type default))
-  )
   (wire (pts (xy 131.572 358.648) (xy 131.572 373.888))
     (stroke (width 0) (type default))
@@
     (stroke (width 0) (type default))
   )
+  (wire (pts (xy 210.566 65.024) (xy 210.566 67.818))
+    (stroke (width 0) (type default))
+  )
   (wire (pts (xy 108.458 118.11) (xy 108.458 123.444))
     (stroke (width 0) (type default))
@@
     (stroke (width 0) (type default))
   )
+  (wire (pts (xy 350.774 48.26) (xy 350.774 51.308))
+    (stroke (width 0) (type default))
+  )
   (wire (pts (xy 188.214 126.238) (xy 188.214 131.826))
     (stroke (width 0) (type default))
@@
     (stroke (width 0) (type default))
   )
-  (wire (pts (xy 221.742 122.174) (xy 210.566 122.174))
+  (wire (pts (xy 221.742 121.92) (xy 210.566 121.92))
     (stroke (width 0) (type default))
   )
@@
     (stroke (width 0) (type default))
   )
+  (wire (pts (xy 221.742 121.92) (xy 221.742 122.174))
+    (stroke (width 0) (type default))
+  )
   (wire (pts (xy 190.5 271.018) (xy 190.5 284.48))
     (stroke (width 0) (type default))
@@
     )
   )
+  (symbol (lib_id "power:-12V") (at 350.774 51.308 180) (unit 1)
+    (in_bom yes) (on_board yes) (dnp no)
+    (property "Reference" "#PWR086" (at 350.774 53.848 0)
+      (effects (font (size 1.27 1.27)) hide)
+    )
+    (property "Value" "-12V" (at 350.52 54.61 0)
+      (effects (font (size 0.75 0.75)))
+    )
+    (property "Footprint" "" (at 350.774 51.308 0)
+      (effects (font (size 1.27 1.27)) hide)
+    )
+    (property "Datasheet" "" (at 350.774 51.308 0)
+      (effects (font (size 1.27 1.27)) hide)
+    )
+    (pin "1")
+    (instances
+      (project "cpu-2"
+        (path "/0d40da8b-082c-404e-8b7d-00a504b0b5d0"
+          (reference "#PWR086") (unit 1)
+        )
+      )
+    )
+  )
   (symbol (lib_id "Sphere:RC42GF131") (at 314.96 229.108 90) (unit 1)
     (in_bom yes) (on_board yes) (dnp no)
@@
         )
       )
+    )
+  )
+  (symbol (lib_id "power:+5V") (at 345.694 51.308 180) (unit 1)
+    (in_bom yes) (on_board yes) (dnp no)
+    (property "Reference" "#PWR085" (at 345.694 47.498 0)
+      (effects (font (size 1.27 1.27)) hide)
+    )
+    (property "Value" "+5V" (at 345.694 54.61 0)
+      (effects (font (size 0.75 0.75)))
+    )
+    (property "Footprint" "" (at 345.694 51.308 0)
+      (effects (font (size 1.27 1.27)) hide)
+    )
+    (property "Datasheet" "" (at 345.694 51.308 0)
+      (effects (font (size 1.27 1.27)) hide)
+    )
+    (pin "1")
+    (instances
+      (project "cpu-2"
+        (path "/0d40da8b-082c-404e-8b7d-00a504b0b5d0"
+          (reference "#PWR085") (unit 1)
+        )
+      )
